File: Fugu2.kicad_sch (KiCad schematic)
At the start: 47 parts, among them J10 691256610002, J3 Conn_L_SW, J6 Conn_L_out, J9 691256610002, Q1 IPA050N10NM5S, Q2 IPP022N12NM6, Q3 IPA050N10NM5S, Q5 TPH1R306PL,L1Q or NTMFS5C612N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, Q6 TPH1R306PL,L1Q or NTMFS5C612N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, Q7 TPH1R306PL,L1Q or NTMFS5C612N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

Commit message: Add project attributions: LICENSE. project name, HW version, Authors
LICENSE: Solderpad Hardware License v2.1
project name: Fugu2
HW version: v2,4
Authors: Fabian, Vadym Vikulin
Other:
- company: (none) -> Fabian (gh@fabi.me), Vadym Vikulin (vadym.vikulin@gmail.com)
- title: (none) -> Fugu2
Changed lines of the file:
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@@
 	(paper "A4")
 	(title_block
+		(title "Fugu2")
 		(date "2026-07-17")
 		(rev "v2.4")
+		(company "Fabian (gh@fabi.me), Vadym Vikulin (vadym.vikulin@gmail.com)")
 	)
 	(rectangle
@@
 	(text "TODO\n- use 2p fuses?\n- extension header 12V, 3.3V, i2c, io pins, SPI?\n   -> UEXT connector (SPI, i2c, UART)\n- LCD and buttons?\n- replace Cin 10u with 4.7u\n- external temp\n"
 		(exclude_from_sim no)
-		(at 179.07 181.61 0)
+		(at 176.784 164.592 0)
 		(effects
 			(font
