File: GateDrive.kicad_sch (KiCad schematic)
At the start: 27 parts, among them Q4 BSS123, U1 UCC21330BQDRQ1

Commit message: Add RC connection between USB-C shield and GND
1. Added a 1 MΩ resistor and 10 nF capacitor between the USB Type-C connector shield and GND in the schematic and PCB layout.
2. Added clearer USB connector symbol having no missing pads
Parts:
- PWRGND1, TPHO1, bfg1, bfs1: value ~ -> (none)

Commit message: Add project attributions: LICENSE. project name, HW version, Authors
LICENSE: Solderpad Hardware License v2.1
project name: Fugu2
HW version: v2,4
Authors: Fabian, Vadym Vikulin
Other:
- company: (none) -> Fabian (gh@fabi.me), Vadym Vikulin (vadym.vikulin@gmail.com)
- title: (none) -> Fugu2
Changed lines of the file:
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@@
 	(paper "A4")
 	(title_block
+		(title "Fugu2")
 		(date "2026-07-17")
 		(rev "v2.4")
+		(company "Fabian (gh@fabi.me), Vadym Vikulin (vadym.vikulin@gmail.com)")
 	)
 	(text "tDT_ns(RDT_kΩ) ≈ 8.6 * RDT_kΩ + 13 \nRDT		tDT\n10k		99ns\n20k		185ns\n50k		443ns \n100k	870ns\n"
