File: PowerSupply.kicad_sch (KiCad schematic)
At the start: 23 parts, among them J7 3.3V PSU, J8 12V PSU, Q8 GT800N10D3, Q9 BSS123, U5 AP3012

Commit message: Add project attributions: LICENSE. project name, HW version, Authors
LICENSE: Solderpad Hardware License v2.1
project name: Fugu2
HW version: v2,4
Authors: Fabian, Vadym Vikulin
Other:
- company: (none) -> Fabian (gh@fabi.me), Vadym Vikulin (vadym.vikulin@gmail.com)
- title: (none) -> Fugu2
Changed lines of the file:
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@@
 	(paper "A4")
 	(title_block
+		(title "Fugu2")
 		(date "2026-07-17")
 		(rev "v2.4")
+		(company "Fabian (gh@fabi.me), Vadym Vikulin (vadym.vikulin@gmail.com)")
 	)
 	(text "Rfb2\n"
