File: Sensors.kicad_sch (KiCad schematic)
At the start: 22 parts, among them U3 INA226, U6 AS333

Commit message: Add project attributions: LICENSE. project name, HW version, Authors
LICENSE: Solderpad Hardware License v2.1
project name: Fugu2
HW version: v2,4
Authors: Fabian, Vadym Vikulin
Other:
- company: (none) -> Fabian (gh@fabi.me), Vadym Vikulin (vadym.vikulin@gmail.com)
- title: (none) -> Fugu2
Changed lines of the file:
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@@
 	(paper "A4")
 	(title_block
+		(title "Fugu2")
 		(date "2026-07-17")
 		(rev "v2.4")
+		(company "Fabian (gh@fabi.me), Vadym Vikulin (vadym.vikulin@gmail.com)")
 	)
 	(text "RC is filter and\ntransient suppressor"
